File: corne-light/pcb/corne-light.kicad_pcb (KiCad board)
At the start: 2 copper layers, 275.5 x 105.6 mm, 122 parts, among them J1 MJ-4PP-9, J2 OLED, J5 Breakaway_Tabs, J6 MJ-4PP-9, J7 OLED, SW1 SW_PUSH, SW10 SW_PUSH, SW11 SW_PUSH, SW12 SW_PUSH, SW13 SW_PUSH, SW14 SW_PUSH, SW15 SW_PUSH, SW16 SW_PUSH, SW17 SW_PUSH, SW18 SW_PUSH, SW19 SW_PUSH, SW2 SW_PUSH, SW20 SW_PUSH, SW21 SW_PUSH, SW22 SW_PUSH, SW23 SW_PUSH, SW24 SW_PUSH, SW25 SW_PUSH, SW26 SW_PUSH, SW27 SW_PUSH, SW28 SW_PUSH, SW29 SW_PUSH, SW3 SW_PUSH, SW30 SW_PUSH, SW31 SW_PUSH, SW32 SW_PUSH, SW33 SW_PUSH, SW34 SW_PUSH, SW35 SW_PUSH, SW36 SW_PUSH, SW37 SW_PUSH, SW38 SW_PUSH, SW39 SW_PUSH, SW4 SW_PUSH, SW40 SW_PUSH, SW41 SW_PUSH, SW42 SW_PUSH, SW5 SW_PUSH, SW6 SW_PUSH, SW7 SW_PUSH, SW8 SW_PUSH, SW9 SW_PUSH, U1 ProMicro, U2 ProMicro

Commit message: Changed stagger of pinky collumns
Parts:
- removed the Ref** at (250.2, 55.4)
- removed the Ref** at (250.2, 74.4)
- removed the Ref** at (50.7, 55.4)
- removed the Ref** at (50.7, 74.4)
- moved D22 8.25 mm to (270.6, 54.2)
- moved D23 8.25 mm to (267.6, 54.2)
- moved J5 8.25 mm to (278.8, 101.6)
- moved Ref** 8.25 mm to (269.2, 63.7)
- moved Ref** 8.25 mm to (269.2, 82.7)
- moved SW22 8.25 mm to (278.6, 54.2)
- moved SW23 8.25 mm to (259.6, 54.2)
- moved D28 8.25 mm to (270.6, 73.2)
- moved D29 8.25 mm to (267.6, 73.2)
- moved D34 8.25 mm to (270.6, 92.2)
- moved D35 8.25 mm to (267.6, 92.2)
- moved SW28 8.25 mm to (278.6, 73.2)
- moved SW29 8.25 mm to (259.6, 73.2)
- moved SW34 8.25 mm to (278.6, 92.2)
- moved SW35 8.25 mm to (259.6, 92.2)
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Routing:
- net col1_r: track 161.3 -> 166.8 mm
- net row2_r: track 137.6 -> 142.9 mm
- net row0: track 142.3 -> 146.2 mm
- net col1: track 156.5 -> 159.9 mm
- net col0: track 182.3 -> 185.7 mm
- net row2: track 153.9 -> 157.2 mm
- net row1_r: track 134.3 -> 137.3 mm
- net col0_r: track 183.2 -> 186.2 mm
- net row0_r: track 127.8 -> 130.5 mm
Other:
- board size 275.5 x 105.6 mm -> 275.5 x 112.7 mm
- net class Default removed
- net class Min removed
