File: corne-light/pcb/corne-light.kicad_pcb (KiCad board)
At the start: 2 copper layers, 275.5 x 112.7 mm, 118 parts, among them J1 MJ-4PP-9, J2 OLED, J5 Breakaway_Tabs, J6 MJ-4PP-9, J7 OLED, SW1 SW_PUSH, SW10 SW_PUSH, SW11 SW_PUSH, SW12 SW_PUSH, SW13 SW_PUSH, SW14 SW_PUSH, SW15 SW_PUSH, SW16 SW_PUSH, SW17 SW_PUSH, SW18 SW_PUSH, SW19 SW_PUSH, SW2 SW_PUSH, SW20 SW_PUSH, SW21 SW_PUSH, SW22 SW_PUSH, SW23 SW_PUSH, SW24 SW_PUSH, SW25 SW_PUSH, SW26 SW_PUSH, SW27 SW_PUSH, SW28 SW_PUSH, SW29 SW_PUSH, SW3 SW_PUSH, SW30 SW_PUSH, SW31 SW_PUSH, SW32 SW_PUSH, SW33 SW_PUSH, SW34 SW_PUSH, SW35 SW_PUSH, SW36 SW_PUSH, SW37 SW_PUSH, SW38 SW_PUSH, SW39 SW_PUSH, SW4 SW_PUSH, SW40 SW_PUSH, SW41 SW_PUSH, SW42 SW_PUSH, SW5 SW_PUSH, SW6 SW_PUSH, SW7 SW_PUSH, SW8 SW_PUSH, SW9 SW_PUSH, U1 ProMicro, U2 ProMicro

Commit message: added artwork
Parts:
- removed the G*** at (60.2, 90.9)
- removed the G*** at (241.0, 91.0)
- removed the G*** at (60.0, 90.9)
- removed the G*** at (240.8, 91.0)
- added G***: LOGO, Thorne:version, F.Cu at (240.8, 89.7)
- added G***: LOGO, Thorne:version, F.Cu at (60.4, 89.7)
- added G***: LOGO, Thorne:background3, F.Cu at (110.8, 33.4)
- added G***: LOGO, Thorne:Version_front, F.Cu at (240.7, 89.7)
- added G***: LOGO, Thorne:Version_front, F.Cu at (60.3, 89.7)
- added G***: LOGO, Thorne:background3_inverted, F.Cu at (206.8, 47.3)
Routing:
- net row1: track 164.3 -> 164.9 mm
Other:
- board text removed: "Corne Light v2.0 PCB Designed by foostan"
